Commit message: launchファイルをv4.5用に変更

File: urdf/my_cugo_robot.urdf.xacro (robot description, xacro)
@@ -2,5 +2,5 @@
 <robot name="my_custom_cugo" xmlns:xacro="http://www.ros.org/wiki/xacro">
   <!-- cugo共通のurdf -->
-  <xacro:include filename="$(find cugo_ros2_control2)/urdf/parts/cugo_base.urdf.xacro" />
+  <xacro:include filename="$(find cugo_ros2_control2)/urdf/parts/cugov4_5_base.urdf.xacro" />
   <xacro:cugo_base />
   <!-- 任意のセンサを追加するurdf -->

File: urdf/parts/cugov4_5_base.urdf.xacro (robot description, xacro)
@@ -18,5 +18,5 @@
     </link>
     <joint name="base_to_left_clawler_joint" type="continuous">
-      <origin xyz="0.0 0.188 0.03835" rpy="0 0 0"/>
+      <origin xyz="0.0 0.190 0.03835" rpy="0 0 0"/>
       <parent link="base_link"/>
       <child link="left_clawler_link"/>
@@ -32,5 +32,5 @@
     </link>
     <joint name="base_to_right_clawler_joint" type="continuous">
-      <origin xyz="0.0 -0.188 0.03835" rpy="0 0 0"/>
+      <origin xyz="0.0 -0.190 0.03835" rpy="0 0 0"/>
       <parent link="base_link"/>
       <child link="right_crawler_link"/>
