Commit message: urdfを修正

File: urdf/parts/cugov4_5_base.urdf.xacro (robot description, xacro)
@@ -3,22 +3,53 @@
   <xacro:macro name="cugo_base">
     <link name="base_footprint" />
-    <link name="base_link" />
+    <link name="base_link">
+      <visual>
+        <geometry>
+          <box size=" 0.590  0.260  0.120"/>
+        </geometry>
+        <origin xyz=" 0.000  0.000 -0.060" rpy="0.000 0.000 0.000"/>
+      </visual>
+      <visual>
+        <geometry>
+          <box size=" 0.165  0.562  0.085"/>
+        </geometry>
+        <origin xyz="-0.2125 0.000  0.0425" rpy="0.000 0.000 0.000"/>
+      </visual>
+      <collision>
+        <geometry>
+          <box size=" 0.590  0.260  0.120"/>
+        </geometry>
+        <origin xyz=" 0.000  0.000 -0.060" rpy="0.000 0.000 0.000"/>
+      </collision>
+      <collision>
+        <geometry>
+          <box size=" 0.165  0.562  0.085"/>
+        </geometry>
+        <origin xyz="-0.2125 0.000  0.0425" rpy="0.000 0.000 0.000"/>
+      </collision>
+    </link>
     <joint name="base_footprint_to_base_link_joint" type="fixed">
       <parent link="base_footprint"/>
       <child link="base_link"/>
-      <origin xyz="0 0 0" rpy="0 0 0" />
+      <origin xyz=" 0.000  0.000  0.170" rpy="0.000 0.000 0.000" />
     </joint>
-    <link name="left_clawler_link">
-       <visual>
+    <link name="left_crawler_link">
+      <visual>
         <geometry>
-          <cylinder radius="0.03835" length="0.07"/>
+          <cylinder radius="0.03835" length="0.120"/>
         </geometry>
-        <origin rpy="1.5707 0 0" xyz="0 0 0"/>
+        <origin rpy="${pi/2} 0.000 0.000" xyz="0.000 0.000 0.000"/>
       </visual>
+      <collision>
+        <geometry>
+          <cylinder radius="0.03835" length="0.120"/>
+        </geometry>
+        <origin rpy="${pi/2} 0.000 0.000" xyz="0.000 0.000 0.000"/>
+      </collision>
     </link>
-    <joint name="base_to_left_clawler_joint" type="continuous">
-      <origin xyz="0.0 0.190 0.03835" rpy="0 0 0"/>
+    <joint name="base_to_left_crawler_joint" type="continuous">
+      <origin xyz="0.000 0.130 -0.13165" rpy="0.000 0.000 0.000"/>
       <parent link="base_link"/>
-      <child link="left_clawler_link"/>
+      <child link="left_crawler_link"/>
       <axis xyz="0 1 0"/>
     </joint>
@@ -26,11 +57,17 @@
       <visual>
         <geometry>
-          <cylinder radius="0.03835" length="0.07"/>
+          <cylinder radius="0.03835" length="0.120"/>
         </geometry>
-        <origin rpy="1.5707 0 0" xyz="0 0 0"/>
+        <origin rpy="${pi/2} 0.000 0.000" xyz="0.000 0.000 0.000"/>
       </visual>
+      <collision>
+        <geometry>
+          <cylinder radius="0.03835" length="0.120"/>
+        </geometry>
+        <origin rpy="${pi/2} 0.000 0.000" xyz="0.000 0.000 0.000"/>
+      </collision>
     </link>
-    <joint name="base_to_right_clawler_joint" type="continuous">
-      <origin xyz="0.0 -0.190 0.03835" rpy="0 0 0"/>
+    <joint name="base_to_right_crawler_joint" type="continuous">
+      <origin xyz="0.000 -0.130 -0.13165" rpy="0.000 0.000 0.000"/>
       <parent link="base_link"/>
       <child link="right_crawler_link"/>
