Commit message: urdfを更新

File: urdf/parts/cugo_v4_5_base.urdf.xacro (robot description, xacro)
@@ -39,5 +39,17 @@
           <cylinder radius="0.03835" length="0.120"/>
         </geometry>
-        <origin rpy="${pi/2} 0.000 0.000" xyz="0.000 0.000 0.000"/>
+        <origin rpy="${pi/2} 0.000 0.000" xyz="-0.255 0.000 0.000"/>
+      </visual>
+      <visual>
+        <geometry>
+          <cylinder radius="0.03835" length="0.120"/>
+        </geometry>
+        <origin rpy="${pi/2} 0.000 0.000" xyz=" 0.000 0.000 0.000"/>
+      </visual>
+      <visual>
+        <geometry>
+          <cylinder radius="0.03835" length="0.120"/>
+        </geometry>
+        <origin rpy="${pi/2} 0.000 0.000" xyz=" 0.255 0.000 0.000"/>
       </visual>
       <collision>
@@ -45,9 +57,21 @@
           <cylinder radius="0.03835" length="0.120"/>
         </geometry>
-        <origin rpy="${pi/2} 0.000 0.000" xyz="0.000 0.000 0.000"/>
+        <origin rpy="${pi/2} 0.000 0.000" xyz="-0.255 0.000 0.000"/>
+      </collision>
+      <collision>
+        <geometry>
+          <cylinder radius="0.03835" length="0.120"/>
+        </geometry>
+        <origin rpy="${pi/2} 0.000 0.000" xyz=" 0.000 0.000 0.000"/>
+      </collision>
+      <collision>
+        <geometry>
+          <cylinder radius="0.03835" length="0.120"/>
+        </geometry>
+        <origin rpy="${pi/2} 0.000 0.000" xyz=" 0.255 0.000 0.000"/>
       </collision>
     </link>
     <joint name="base_to_left_crawler_joint" type="continuous">
-      <origin xyz="0.000 0.130 -0.13165" rpy="0.000 0.000 0.000"/>
+      <origin xyz="0.000 0.215 -0.13165" rpy="0.000 0.000 0.000"/>
       <parent link="base_link"/>
       <child link="left_crawler_link"/>
@@ -59,5 +83,17 @@
           <cylinder radius="0.03835" length="0.120"/>
         </geometry>
-        <origin rpy="${pi/2} 0.000 0.000" xyz="0.000 0.000 0.000"/>
+        <origin rpy="${pi/2} 0.000 0.000" xyz="-0.255 0.000 0.000"/>
+      </visual>
+      <visual>
+        <geometry>
+          <cylinder radius="0.03835" length="0.120"/>
+        </geometry>
+        <origin rpy="${pi/2} 0.000 0.000" xyz=" 0.000 0.000 0.000"/>
+      </visual>
+      <visual>
+        <geometry>
+          <cylinder radius="0.03835" length="0.120"/>
+        </geometry>
+        <origin rpy="${pi/2} 0.000 0.000" xyz=" 0.255 0.000 0.000"/>
       </visual>
       <collision>
@@ -65,9 +101,21 @@
           <cylinder radius="0.03835" length="0.120"/>
         </geometry>
-        <origin rpy="${pi/2} 0.000 0.000" xyz="0.000 0.000 0.000"/>
+        <origin rpy="${pi/2} 0.000 0.000" xyz="-0.255 0.000 0.000"/>
+      </collision>
+      <collision>
+        <geometry>
+          <cylinder radius="0.03835" length="0.120"/>
+        </geometry>
+        <origin rpy="${pi/2} 0.000 0.000" xyz=" 0.000 0.000 0.000"/>
+      </collision>
+      <collision>
+        <geometry>
+          <cylinder radius="0.03835" length="0.120"/>
+        </geometry>
+        <origin rpy="${pi/2} 0.000 0.000" xyz=" 0.255 0.000 0.000"/>
       </collision>
     </link>
     <joint name="base_to_right_crawler_joint" type="continuous">
-      <origin xyz="0.000 -0.130 -0.13165" rpy="0.000 0.000 0.000"/>
+      <origin xyz="0.000 -0.215 -0.13165" rpy="0.000 0.000 0.000"/>
       <parent link="base_link"/>
       <child link="right_crawler_link"/>

Commit message: クローラの関係性に誤りがあったので修正

File: urdf/parts/cugo_v4_5_base.urdf.xacro (robot description, xacro)
@@ -34,11 +34,6 @@
       <origin xyz=" 0.000  0.000  0.170" rpy="0.000 0.000 0.000" />
     </joint>
+    <!-- left crawler (center) -->
     <link name="left_crawler_link">
-      <visual>
-        <geometry>
-          <cylinder radius="0.03835" length="0.120"/>
-        </geometry>
-        <origin rpy="${pi/2} 0.000 0.000" xyz="-0.255 0.000 0.000"/>
-      </visual>
       <visual>
         <geometry>
@@ -47,16 +42,4 @@
         <origin rpy="${pi/2} 0.000 0.000" xyz=" 0.000 0.000 0.000"/>
       </visual>
-      <visual>
-        <geometry>
-          <cylinder radius="0.03835" length="0.120"/>
-        </geometry>
-        <origin rpy="${pi/2} 0.000 0.000" xyz=" 0.255 0.000 0.000"/>
-      </visual>
-      <collision>
-        <geometry>
-          <cylinder radius="0.03835" length="0.120"/>
-        </geometry>
-        <origin rpy="${pi/2} 0.000 0.000" xyz="-0.255 0.000 0.000"/>
-      </collision>
       <collision>
         <geometry>
@@ -64,10 +47,4 @@
         </geometry>
         <origin rpy="${pi/2} 0.000 0.000" xyz=" 0.000 0.000 0.000"/>
-      </collision>
-      <collision>
-        <geometry>
-          <cylinder radius="0.03835" length="0.120"/>
-        </geometry>
-        <origin rpy="${pi/2} 0.000 0.000" xyz=" 0.255 0.000 0.000"/>
       </collision>
     </link>
@@ -78,11 +55,46 @@
       <axis xyz="0 1 0"/>
     </joint>
-    <link name="right_crawler_link">
+    <!-- left crawler (front: x=-0.255 in crawler frame → base_link frame) -->
+    <link name="left_front_crawler_link">
       <visual>
         <geometry>
           <cylinder radius="0.03835" length="0.120"/>
         </geometry>
-        <origin rpy="${pi/2} 0.000 0.000" xyz="-0.255 0.000 0.000"/>
+        <origin rpy="${pi/2} 0.000 0.000" xyz="0.000 0.000 0.000"/>
       </visual>
+      <collision>
+        <geometry>
+          <cylinder radius="0.03835" length="0.120"/>
+        </geometry>
+        <origin rpy="${pi/2} 0.000 0.000" xyz="0.000 0.000 0.000"/>
+      </collision>
+    </link>
+    <joint name="base_to_left_front_crawler_joint" type="fixed">
+      <origin xyz="-0.255  0.215 -0.13165" rpy="0.000 0.000 0.000"/>
+      <parent link="base_link"/>
+      <child link="left_front_crawler_link"/>
+    </joint>
+    <!-- left crawler (rear: x=+0.255 in crawler frame → base_link frame) -->
+    <link name="left_rear_crawler_link">
+      <visual>
+        <geometry>
+          <cylinder radius="0.03835" length="0.120"/>
+        </geometry>
+        <origin rpy="${pi/2} 0.000 0.000" xyz="0.000 0.000 0.000"/>
+      </visual>
+      <collision>
+        <geometry>
+          <cylinder radius="0.03835" length="0.120"/>
+        </geometry>
+        <origin rpy="${pi/2} 0.000 0.000" xyz="0.000 0.000 0.000"/>
+      </collision>
+    </link>
+    <joint name="base_to_left_rear_crawler_joint" type="fixed">
+      <origin xyz=" 0.255  0.215 -0.13165" rpy="0.000 0.000 0.000"/>
+      <parent link="base_link"/>
+      <child link="left_rear_crawler_link"/>
+    </joint>
+    <!-- right crawler (center) -->
+    <link name="right_crawler_link">
       <visual>
         <geometry>
@@ -91,16 +103,4 @@
         <origin rpy="${pi/2} 0.000 0.000" xyz=" 0.000 0.000 0.000"/>
       </visual>
-      <visual>
-        <geometry>
-          <cylinder radius="0.03835" length="0.120"/>
-        </geometry>
-        <origin rpy="${pi/2} 0.000 0.000" xyz=" 0.255 0.000 0.000"/>
-      </visual>
-      <collision>
-        <geometry>
-          <cylinder radius="0.03835" length="0.120"/>
-        </geometry>
-        <origin rpy="${pi/2} 0.000 0.000" xyz="-0.255 0.000 0.000"/>
-      </collision>
       <collision>
         <geometry>
@@ -108,10 +108,4 @@
         </geometry>
         <origin rpy="${pi/2} 0.000 0.000" xyz=" 0.000 0.000 0.000"/>
-      </collision>
-      <collision>
-        <geometry>
-          <cylinder radius="0.03835" length="0.120"/>
-        </geometry>
-        <origin rpy="${pi/2} 0.000 0.000" xyz=" 0.255 0.000 0.000"/>
       </collision>
     </link>
@@ -122,4 +116,44 @@
       <axis xyz="0 1 0"/>
     </joint>
+    <!-- right crawler (front: x=-0.255 in crawler frame → base_link frame) -->
+    <link name="right_front_crawler_link">
+      <visual>
+        <geometry>
+          <cylinder radius="0.03835" length="0.120"/>
+        </geometry>
+        <origin rpy="${pi/2} 0.000 0.000" xyz="0.000 0.000 0.000"/>
+      </visual>
+      <collision>
+        <geometry>
+          <cylinder radius="0.03835" length="0.120"/>
+        </geometry>
+        <origin rpy="${pi/2} 0.000 0.000" xyz="0.000 0.000 0.000"/>
+      </collision>
+    </link>
+    <joint name="base_to_right_front_crawler_joint" type="fixed">
+      <origin xyz="-0.255 -0.215 -0.13165" rpy="0.000 0.000 0.000"/>
+      <parent link="base_link"/>
+      <child link="right_front_crawler_link"/>
+    </joint>
+    <!-- right crawler (rear: x=+0.255 in crawler frame → base_link frame) -->
+    <link name="right_rear_crawler_link">
+      <visual>
+        <geometry>
+          <cylinder radius="0.03835" length="0.120"/>
+        </geometry>
+        <origin rpy="${pi/2} 0.000 0.000" xyz="0.000 0.000 0.000"/>
+      </visual>
+      <collision>
+        <geometry>
+          <cylinder radius="0.03835" length="0.120"/>
+        </geometry>
+        <origin rpy="${pi/2} 0.000 0.000" xyz="0.000 0.000 0.000"/>
+      </collision>
+    </link>
+    <joint name="base_to_right_rear_crawler_joint" type="fixed">
+      <origin xyz=" 0.255 -0.215 -0.13165" rpy="0.000 0.000 0.000"/>
+      <parent link="base_link"/>
+      <child link="right_rear_crawler_link"/>
+    </joint>
   </xacro:macro>
 </robot>
